Commit message: modified laser angles

File: car_demo/prius_description/urdf/prius.urdf (robot description, URDF)
Before this commit: robot prius, 24 links, 23 joints
Joints:
- joint front_left_laser_joint: origin xyz=1 -2.3 0.5 rpy=0 0.05 0 -> xyz=1 -2.3 0.5 rpy=0 0.0 0
- joint front_right_laser_joint: origin xyz=-1 -2.3 0.5 rpy=0 0.05 3.14 -> xyz=-1 -2.3 0.5 rpy=0 0.0 3.14
