Commit message: added the correct bmw mesh

File: car_demo/bmw_description/urdf/bmw.urdf (robot description, URDF)
Before this commit: robot bmw, 24 links, 23 joints
Links:
- link chassis: geometry collision box size=1.168381 1.654253 0.272347; collision box size=1.267845 1.116344 0.244286
- link front_left_wheel: geometry collision sphere radius=0.33; visual mesh filename=package://bmw_description/meshes/right_rear_gray.dae scale=1 1 1
- link front_right_wheel: geometry collision sphere radius=0.33; visual mesh filename=package://bmw_description/meshes/right_rear_gray.dae scale=1 1 1
- link rear_left_wheel: geometry collision sphere radius=0.33; visual mesh filename=package://bmw_description/meshes/right_rear_gray.dae scale=1 1 1
- link rear_right_wheel: geometry collision sphere radius=0.33; visual mesh filename=package://bmw_description/meshes/right_rear_gray.dae scale=1 1 1
Joints:
- joint front_left_steer_joint: origin xyz=0.767 -1.41 0.3 rpy=0 0 0 -> xyz=0.767 -1.41 0.2 rpy=0 0 0
- joint front_right_steer_joint: origin xyz=-0.767 -1.41 0.3 rpy=0 0 0 -> xyz=-0.767 -1.41 0.2 rpy=0 0 0
- joint rear_left_wheel_joint: origin xyz=0.793 1.45 0.3 rpy=0 0 0 -> xyz=0.793 1.45 0.2 rpy=0 0 0
- joint rear_right_wheel_joint: origin xyz=-0.793 1.45 0.3 rpy=0 0 0 -> xyz=-0.793 1.45 0.2 rpy=0 0 0
- joint steering_joint: origin xyz=0.357734 -0.627868 0.988243 rpy=-1.302101 0 0 -> xyz=0.4 -0.27 0.72 rpy=-1.302101 0 0
